Commit message: add the manipulation of UR using moveit and gazebo

File: src/tinker_description/urdf/inc/base_macro_display.xacro (robot description, xacro)
@@ -2,16 +2,16 @@
 <robot xmlns:xacro="http://www.ros.org/wiki/xacro" >
   <!-- Due to the different rules for mesh search in gazebo and rviz2, two xacro files are created to designate mesh path -->
-    <xacro:property name="stl_path" value="$(find tinker_sim)/meshes/tinker_base_coarse.stl" />
+    <xacro:property name="stl_path" value="package://tinker_description/meshes/tinker_base_coarse.stl" />
     <xacro:macro name="steering_link_visual_mesh" params="name">
-        <mesh filename="$(find tinker_sim)/meshes/DAE/suspension/${name}_link.dae"/>
+        <mesh filename="package://tinker_description/meshes/DAE/suspension/${name}_link.dae"/>
     </xacro:macro>
     <xacro:macro name="steering_link_collision_mesh">
-        <mesh filename="$(find tinker_sim)/meshes/STL/suspension/sus_link.stl"/>
+        <mesh filename="package://tinker_description/meshes/STL/suspension/sus_link.stl"/>
     </xacro:macro>
     <xacro:macro name="wheel_link_visual_mesh">
-        <mesh filename="$(find tinker_sim)/meshes/DAE/wheel/wheel_link.dae"/>
+        <mesh filename="package://tinker_description/meshes/DAE/wheel/wheel_link.dae"/>
     </xacro:macro>
     <xacro:macro name="wheel_link_collision_mesh">
-        <mesh filename="$(find tinker_sim)/meshes/STL/wheel/robot_wheel.stl"/>
+        <mesh filename="package://tinker_description/meshes/STL/wheel/robot_wheel.stl"/>
     </xacro:macro>
 </robot>

File: src/tinker_description/urdf/inc/base_macro_gazebo.xacro (robot description, xacro)
@@ -2,16 +2,16 @@
 <robot xmlns:xacro="http://www.ros.org/wiki/xacro" >
   <!-- Due to the different rules for mesh search in gazebo and rviz2, two xacro files are created to designate mesh path -->
-    <xacro:property name="stl_path" value="package://tinker_sim/meshes/tinker_base_coarse.stl" />
+    <xacro:property name="stl_path" value="$(find tinker_description)/meshes/tinker_base_coarse.stl" />
     <xacro:macro name="steering_link_visual_mesh" params="name">
-        <mesh filename="package://tinker_sim/meshes/DAE/suspension/${name}_link.dae"/>
+        <mesh filename="$(find tinker_description)/meshes/DAE/suspension/${name}_link.dae"/>
     </xacro:macro>
     <xacro:macro name="steering_link_collision_mesh">
-        <mesh filename="package://tinker_sim/meshes/STL/suspension/sus_link.stl"/>
+        <mesh filename="$(find tinker_description)/meshes/STL/suspension/sus_link.stl"/>
     </xacro:macro>
     <xacro:macro name="wheel_link_visual_mesh">
-        <mesh filename="package://tinker_sim/meshes/DAE/wheel/wheel_link.dae"/>
+        <mesh filename="$(find tinker_description)/meshes/DAE/wheel/wheel_link.dae"/>
     </xacro:macro>
     <xacro:macro name="wheel_link_collision_mesh">
-        <mesh filename="package://tinker_sim/meshes/STL/wheel/robot_wheel.stl"/>
+        <mesh filename="$(find tinker_description)/meshes/STL/wheel/robot_wheel.stl"/>
     </xacro:macro>
 </robot>
