Commit message: add camera to base transform

File: src/tinker_description/urdf/tinker_arm.urdf.xacro (robot description, xacro)
@@ -99,3 +99,9 @@
     <origin xyz="0 0 0.2" />
   </joint>
+  <link name="wrist_camera" />
+  <joint name="camera_to_wrist" type="fixed">
+    <parent link="$(arg prefix)wrist_3_link" />
+    <child link="wrist_camera" />
+    <origin xyz="0 -0.07 -0.025"/>
+  </joint>
 </robot>

File: src/tinker_description/urdf/tinker_gazebo.urdf.xacro (robot description, xacro)
@@ -135,4 +135,7 @@
             <parameters>$(find tinker_sim)/config/tinker_controller_manager.yaml</parameters>
         </plugin>
+        <plugin name="joint_state_publisher" filename="libgazebo_ros_joint_state_publisher.so">
+            <jointName>left_wheel,right_wheel</jointName>
+        </plugin>
     </gazebo>
     <ros2_control name="GazeboSystem" type="system">
