Commit message: fix controller manager does not exit bug

File: src/tinker_description/srdf/ur_macro.srdf.xacro (robot description, xacro)
@@ -12,5 +12,5 @@
     <!--SUBGROUPS - Groups can also be formed by referencing to already defined group names-->
     <group name="${prefix}manipulator">
-      <chain base_link="${prefix}base_link" tip_link="${prefix}tool0" />
+      <chain base_link="${prefix}base_link" tip_link="gripper" />
     </group>
     <!--GROUP STATES - Purpose - Define a named state for a particular group, in terms of joint values. This is useful to define states like 'folded arms'-->

File: src/tinker_description/urdf/tinker_arm.urdf.xacro (robot description, xacro)
@@ -7,4 +7,5 @@
    <!-- To fix the broken joints problem, edit the initial ur_macro.xacro -->
    <xacro:include filename="inc/ur_macro.xacro"/>
+   <xacro:include filename="inc/robotiq_arg2f_140_model_macro.xacro" />
    <!-- possible 'ur_type' values: ur3, ur3e, ur5, ur5e, ur10, ur10e, ur16e -->
    <!-- the default value should raise an error in case this was called without defining the type -->
@@ -12,8 +13,9 @@
    <!-- parameters -->
    <xacro:arg name="tf_prefix" default="ur_" />
-   <xacro:arg name="joint_limit_params" default="$(find ur_description)/config/$(arg ur_type)/joint_limits.yaml"/>
-   <xacro:arg name="kinematics_params" default="$(find ur_description)/config/$(arg ur_type)/default_kinematics.yaml"/>
-   <xacro:arg name="physical_params" default="$(find ur_description)/config/$(arg ur_type)/physical_parameters.yaml"/>
-   <xacro:arg name="visual_params" default="$(find ur_description)/config/$(arg ur_type)/visual_parameters.yaml"/>
+   <xacro:arg name="prefix" default="ur_" />
+   <xacro:arg name="joint_limit_params" default="$(find tinker_description)/config/$(arg ur_type)/joint_limits.yaml"/>
+   <xacro:arg name="kinematics_params" default="$(find tinker_description)/config/$(arg ur_type)/default_kinematics.yaml"/>
+   <xacro:arg name="physical_params" default="$(find tinker_description)/config/$(arg ur_type)/physical_parameters.yaml"/>
+   <xacro:arg name="visual_params" default="$(find tinker_description)/config/$(arg ur_type)/visual_parameters.yaml"/>
    <xacro:arg name="transmission_hw_interface" default=""/>
    <xacro:arg name="safety_limits" default="true"/>
@@ -52,5 +54,5 @@
      name="$(arg name)"
      tf_prefix="$(arg tf_prefix)"
-     parent="tinker"
+     parent="base_link"
      joint_limits_parameters_file="$(arg joint_limit_params)"
      kinematics_parameters_file="$(arg kinematics_params)"
@@ -85,22 +87,15 @@
      <origin xyz="0.1 0 0.64" rpy="0 0 0" />          <!-- position robot on tinker base-->
    </xacro:ur_robot>
-   <!-- <xacro:if value="$(arg sim_gazebo)">
-    <gazebo reference="world">
-    </gazebo>
-    <gazebo>
-      <plugin filename="libgazebo_ros2_control.so" name="gazebo_ros2_control">
-        <parameters>$(arg simulation_controllers)</parameters>
-      </plugin>
-    </gazebo>
-  </xacro:if> -->
-  <!-- <xacro:if value="$(arg sim_ignition)">
-    <gazebo reference="world">
-    </gazebo>
-    <gazebo>
-      <plugin filename="libign_ros2_control-system.so" name="ign_ros2_control::IgnitionROS2ControlPlugin">
-        <parameters>$(arg simulation_controllers)</parameters>
-        <controller_manager_node_name>$(arg tf_prefix)controller_manager</controller_manager_node_name>
-      </plugin>
-    </gazebo>
-  </xacro:if> -->
+  <xacro:robotiq_arg2f_140 prefix="$(arg prefix)"/>
+  <joint name="arm_to_finger" type="fixed">
+    <parent link="$(arg tf_prefix)tool0" />
+    <child link="$(arg prefix)robotiq_arg2f_base_link" />
+    <origin xyz="0 0 0" />
+  </joint>
+  <link name="gripper" />
+  <joint name="middle_of_finger_pad" type="fixed">
+    <parent link="$(arg prefix)robotiq_arg2f_base_link" />
+    <child link="gripper" />
+    <origin xyz="0 0 0" />
+  </joint>
 </robot>

Commit message: moveit control with gripper urdf added

File: src/tinker_description/srdf/ur_macro.srdf.xacro (robot description, xacro)
@@ -53,4 +53,19 @@
     <disable_collisions link1="${prefix}wrist_1_link" link2="${prefix}wrist_3_link" reason="Never" />
     <disable_collisions link1="${prefix}wrist_2_link" link2="${prefix}wrist_3_link" reason="Adjacent" />
+    <disable_collisions link1="${prefix}robotiq_arg2f_base_link" link2="${prefix}wrist_3_link" reason="Adjacent" />
+    <disable_collisions link1="${prefix}left_inner_finger" link2="${prefix}left_inner_finger_pad" reason="Adjacent" />
+    <disable_collisions link1="${prefix}left_inner_finger" link2="${prefix}left_inner_knuckle" reason="Adjacent" />
+    <disable_collisions link1="${prefix}left_inner_finger" link2="${prefix}left_outer_finger" reason="Adjacent" />
+    <disable_collisions link1="${prefix}left_outer_knuckle" link2="${prefix}left_inner_knuckle" reason="Adjacent" />
+    <disable_collisions link1="${prefix}left_outer_knuckle" link2="${prefix}left_outer_finger" reason="Adjacent" />
+    <disable_collisions link1="${prefix}left_outer_knuckle" link2="${prefix}robotiq_arg2f_base_link" reason="Adjacent" />
+    <disable_collisions link1="${prefix}left_inner_knuckle" link2="${prefix}robotiq_arg2f_base_link" reason="Adjacent" />
+    <disable_collisions link1="${prefix}right_inner_finger" link2="${prefix}right_inner_finger_pad" reason="Adjacent" />
+    <disable_collisions link1="${prefix}right_inner_finger" link2="${prefix}right_outer_finger" reason="Adjacent" />
+    <disable_collisions link1="${prefix}right_inner_finger" link2="${prefix}right_inner_knuckle" reason="Adjacent" />
+    <disable_collisions link1="${prefix}right_outer_knuckle" link2="${prefix}right_inner_knuckle" reason="Adjacent" />
+    <disable_collisions link1="${prefix}right_outer_knuckle" link2="${prefix}right_outer_finger" reason="Adjacent" />
+    <disable_collisions link1="${prefix}right_outer_knuckle" link2="${prefix}robotiq_arg2f_base_link" reason="Adjacent" />
+    <disable_collisions link1="${prefix}right_inner_knuckle" link2="${prefix}robotiq_arg2f_base_link" reason="Adjacent" />
   </xacro:macro>
 </robot>

File: src/tinker_description/urdf/tinker_arm.urdf.xacro (robot description, xacro)
@@ -97,5 +97,5 @@
     <parent link="$(arg prefix)robotiq_arg2f_base_link" />
     <child link="gripper" />
-    <origin xyz="0 0 0" />
+    <origin xyz="0 0 0.2" />
   </joint>
 </robot>

Commit message: grasp debug

File: src/tinker_description/srdf/ur_macro.srdf.xacro (robot description, xacro)
@@ -31,11 +31,11 @@
       <joint name="${prefix}wrist_3_joint" value="0" />
     </group_state>
-    <group_state name="${prefix}test_configuration" group="${prefix}manipulator">
-      <joint name="${prefix}elbow_joint" value="1.4" />
-      <joint name="${prefix}shoulder_lift_joint" value="-1.62" />
-      <joint name="${prefix}shoulder_pan_joint" value="1.54" />
-      <joint name="${prefix}wrist_1_joint" value="-1.2" />
-      <joint name="${prefix}wrist_2_joint" value="-1.6" />
-      <joint name="${prefix}wrist_3_joint" value="-0.11" />
+    <group_state name="${prefix}grasp_initial" group="${prefix}manipulator">
+      <joint name="${prefix}elbow_joint" value="-0.785" />
+      <joint name="${prefix}shoulder_lift_joint" value="-1.22" />
+      <joint name="${prefix}shoulder_pan_joint" value="-2.35" />
+      <joint name="${prefix}wrist_1_joint" value="-2.1" />
+      <joint name="${prefix}wrist_2_joint" value="-4.65" />
+      <joint name="${prefix}wrist_3_joint" value="0." />
     </group_state>
     <!--END EFFECTOR - Purpose - Represent information about an end effector.-->
@@ -68,4 +68,5 @@
     <disable_collisions link1="${prefix}right_outer_knuckle" link2="${prefix}robotiq_arg2f_base_link" reason="Adjacent" />
     <disable_collisions link1="${prefix}right_inner_knuckle" link2="${prefix}robotiq_arg2f_base_link" reason="Adjacent" />
+    <disable_collisions link1="realsense" link2="${prefix}wrist_3_link" reason="Adjacent" />
   </xacro:macro>
 </robot>

File: src/tinker_description/urdf/tinker_arm.urdf.xacro (robot description, xacro)
@@ -85,5 +85,5 @@
      script_command_port="$(arg script_command_port)"
      >
-     <origin xyz="0.1 0 0.64" rpy="0 0 0" />          <!-- position robot on tinker base-->
+     <origin xyz="0.1 0 0.64" rpy="0 0 -0.785" />          <!-- position robot on tinker base-->
    </xacro:ur_robot>
   <xacro:robotiq_arg2f_140 prefix="$(arg prefix)"/>
@@ -91,5 +91,5 @@
     <parent link="$(arg tf_prefix)tool0" />
     <child link="$(arg prefix)robotiq_arg2f_base_link" />
-    <origin xyz="0 0 0" />
+    <origin xyz="0 0 0" rpy="0 0 1.57"/>
   </joint>
   <link name="gripper" />
@@ -103,5 +103,22 @@
     <parent link="$(arg prefix)wrist_3_link" />
     <child link="wrist_camera" />
-    <origin xyz="0 -0.07 -0.025"/>
+    <origin xyz="0 -0.08 -0.025"/>
+  </joint>
+  <link name="realsense">
+    <visual>
+      <geometry>
+       <box size="0.1 0.04 0.02"/>
+      </geometry>
+    </visual>
+    <collision>
+      <geometry>
+       <box size="0.1 0.04 0.02"/>
+      </geometry>
+    </collision>
+  </link>
+  <joint name="fix_realsense" type="fixed">
+    <parent link="wrist_camera" />
+    <child link="realsense" />
+    <origin xyz="0. 0.02 0." />
   </joint>
 </robot>

File: src/tinker_description/urdf/tinker_base.urdf.xacro (robot description, xacro)
@@ -121,5 +121,5 @@
     </link>
   </xacro:macro>
-  <xacro:susp_gen name="fl" prefix_1="1" prefix_2="1" />
+  <!-- <xacro:susp_gen name="fl" prefix_1="1" prefix_2="1" />
   <xacro:wheel_gen name="fl" prefix_1="1" prefix_2="1" />
   <xacro:susp_gen name="fr" prefix_1="1" prefix_2="-1" />
@@ -128,4 +128,4 @@
   <xacro:wheel_gen name="rl" prefix_1="-1" prefix_2="1" />
   <xacro:susp_gen name="rr" prefix_1="-1" prefix_2="-1" />
-  <xacro:wheel_gen name="rr" prefix_1="-1" prefix_2="-1" />
+  <xacro:wheel_gen name="rr" prefix_1="-1" prefix_2="-1" /> -->
 </robot>

File: src/tinker_description/urdf/tinker_gazebo.urdf.xacro (robot description, xacro)
@@ -139,5 +139,5 @@
         </plugin>
     </gazebo>
-    <ros2_control name="GazeboSystem" type="system">
+    <!-- <ros2_control name="GazeboSystem" type="system">
         <hardware>
             <plugin>gazebo_ros2_control/GazeboSystem</plugin>
@@ -151,4 +151,4 @@
         <xacro:steering_interface name="rl"/>
         <xacro:steering_interface name="rr"/>
-    </ros2_control>
+    </ros2_control> -->
 </robot>

Commit message: add realsense urdf

File: src/tinker_description/srdf/ur_macro.srdf.xacro (robot description, xacro)
@@ -68,5 +68,5 @@
     <disable_collisions link1="${prefix}right_outer_knuckle" link2="${prefix}robotiq_arg2f_base_link" reason="Adjacent" />
     <disable_collisions link1="${prefix}right_inner_knuckle" link2="${prefix}robotiq_arg2f_base_link" reason="Adjacent" />
-    <disable_collisions link1="realsense" link2="${prefix}wrist_3_link" reason="Adjacent" />
+    <disable_collisions link1="wrist" link2="${prefix}wrist_3_link" reason="Adjacent" />
   </xacro:macro>
 </robot>

File: src/tinker_description/urdf/inc/realsense/_d435i.urdf.xacro (robot description, xacro)
@@ -19,8 +19,8 @@
 aluminum peripherial evaluation case.
 -->
-<robot xmlns:xacro="http://ros.org/wiki/xacro">
-  <xacro:include filename="realsense/_d435.urdf.xacro"/>
-  <xacro:include filename="realsense/_d435i_imu_modules.urdf.xacro"/>
-  <xacro:macro name="realsense" params="parent *origin name:=camera use_nominal_extrinsics:=false">
+<robot name="sensor_d435i" xmlns:xacro="http://ros.org/wiki/xacro">
+  <xacro:include filename="$(find realsense2_description)/urdf/_d435.urdf.xacro"/>
+  <xacro:include filename="$(find realsense2_description)/urdf/_d435i_imu_modules.urdf.xacro"/>
+  <xacro:macro name="sensor_d435i" params="parent *origin name:=camera use_nominal_extrinsics:=false">
     <xacro:sensor_d435 parent="${parent}" name="${name}" use_nominal_extrinsics="${use_nominal_extrinsics}">
       <xacro:insert_block name="origin" />

File: src/tinker_description/urdf/inc/realsense/_materials.urdf.xacro (robot description, xacro)
@@ -16,15 +16,17 @@
 -->
 <!--
-This is the URDF model for the Intel RealSense 435i camera, in it's
-aluminum peripherial evaluation case.
+Collection of materials to be used in other macros.
+This avoids the redefinition of materials in case multple cameras are imported.
 -->
 <robot xmlns:xacro="http://ros.org/wiki/xacro">
-  <xacro:include filename="realsense/_d435.urdf.xacro"/>
-  <xacro:include filename="realsense/_d435i_imu_modules.urdf.xacro"/>
-  <xacro:macro name="realsense" params="parent *origin name:=camera use_nominal_extrinsics:=false">
-    <xacro:sensor_d435 parent="${parent}" name="${name}" use_nominal_extrinsics="${use_nominal_extrinsics}">
-      <xacro:insert_block name="origin" />
-    </xacro:sensor_d435>
-    <xacro:d435i_imu_modules name="${name}" use_nominal_extrinsics="${use_nominal_extrinsics}"/>
-  </xacro:macro>
+  <xacro:property name="realsense_materials_defined" default="false" />
+  <xacro:unless value="${realsense_materials_defined}">
+    <xacro:property name="realsense_materials_defined" value="true" />
+    <material name="aluminum">
+      <color rgba="0.5 0.5 0.5 1"/>
+    </material>
+    <material name="plastic">
+      <color rgba="0.1 0.1 0.1 1"/>
+    </material>
+ </xacro:unless>
 </robot>

File: src/tinker_description/urdf/tinker_arm.urdf.xacro (robot description, xacro)
@@ -8,5 +8,5 @@
    <xacro:include filename="inc/ur_macro.xacro"/>
    <xacro:include filename="inc/robotiq_arg2f_140_model_macro.xacro" />
-   <!-- <xacro:include filename="inc/_d435i.urdf.xacro" /> -->
+   <xacro:include filename="inc/_d435i.urdf.xacro" />
    <!-- possible 'ur_type' values: ur3, ur3e, ur5, ur5e, ur10, ur10e, ur16e -->
    <!-- the default value should raise an error in case this was called without defining the type -->
@@ -98,28 +98,27 @@
     <parent link="$(arg prefix)robotiq_arg2f_base_link" />
     <child link="gripper" />
-    <origin xyz="0 0 0.2" />
+    <origin xyz="0 0 0.22" />
   </joint>
-  <link name="wrist_camera" />
-  <joint name="camera_to_wrist" type="fixed">
-    <parent link="$(arg prefix)wrist_3_link" />
-    <child link="wrist_camera" />
-    <origin xyz="0 -0.08 -0.025"/>
-  </joint>
-  <link name="realsense">
+ <link name="wrist">
     <visual>
       <geometry>
-       <box size="0.1 0.04 0.02"/>
+        <mesh filename="file://$(find tinker_description)/meshes/wrist.STL" scale="0.001 0.001 0.001"/>
       </geometry>
+      <material name="white"/>
     </visual>
     <collision>
       <geometry>
-       <box size="0.1 0.04 0.02"/>
+        <mesh filename="file://$(find tinker_description)/meshes/wrist.STL" scale="0.001 0.001 0.001"/>
       </geometry>
     </collision>
   </link>
-  <joint name="fix_realsense" type="fixed">
-    <parent link="wrist_camera" />
-    <child link="realsense" />
-    <origin xyz="0. 0.02 0." />
+  <joint name="wrist_to_ur" type="fixed">
+    <parent link="$(arg prefix)tool0" />
+    <child link="wrist" />
+    <origin xyz="0.068 0.048 0.0" rpy="0 3.1415926 1.5708"/>
   </joint>
+  <xacro:realsense
+    parent="$(arg tf_prefix)tool0">
+    <origin xyz="0 -0.07 -0.015" rpy="0 -1.5708 1.5708" />          <!-- the result of calibration -->
+   </xacro:realsense>
 </robot>

Commit message: update urdf

File: src/tinker_description/srdf/ur_macro.srdf.xacro (robot description, xacro)
@@ -69,4 +69,5 @@
     <disable_collisions link1="${prefix}right_inner_knuckle" link2="${prefix}robotiq_arg2f_base_link" reason="Adjacent" />
     <disable_collisions link1="wrist" link2="${prefix}wrist_3_link" reason="Adjacent" />
+    <disable_collisions link1="wrist" link2="camera_link" reason="Adjacent" />
   </xacro:macro>
 </robot>

File: src/tinker_description/urdf/tinker_arm.urdf.xacro (robot description, xacro)
@@ -120,5 +120,5 @@
   <xacro:realsense
     parent="$(arg tf_prefix)tool0">
-    <origin xyz="0 -0.07 -0.015" rpy="0 -1.5708 1.5708" />          <!-- the result of calibration -->
+    <origin xyz="-0.009067 -0.060051 -0.013648" rpy="0.0268678 -1.5471549 1.5684374" />          <!-- the result of calibration -->
    </xacro:realsense>
 </robot>
